File: nephelometer/circuitry/band psd v1.1 shield.sch (EAGLE design)
At the start: 57 parts, among them IC1 LMC6484P, IC2 LM555N, IC3 74HCT74N, IC4 4044N, T1 2N2222, T2 2N2222, U1 MAX4544, U4 MotA

Commit message: Updated to use MCP3301 for ADC on stand-alone
Parts:
- added C16: 100n, adafruit:C-US025-025X050
- added IC5: (no value), ingolia:MCP3301
Connections:
- new net CS_ADC: IC5.SHDN, U3.A2
- new net MISO: IC5.DOUT, U3.MISO
- new net SCK: IC5.CLK, U3.SCK
- net +5V: now also C16.1, IC5.VDD
- net 2.5V: now also IC5.IN+, IC5.VREF; no longer U3.A4, U3.AREF
- net GND: now also C16.2, IC5.GND
- net N$28: now also IC5.IN-; no longer U3.A5
Other:
- note added: "5kHz clock low => LED ON => TIA output higher to raise (-) voltage => 10x BP output lower to reduce (-) voltage => inverter output higher to raise (-) voltage 5kHz low => N.C. [lower in LED ON] selected 5kHz higher => N.O. [lower in LED OFF] selected SO output always lower"
- moved on the sheet: C14, Q3, U2
