File: nephelometer/circuitry/band-psd-micro-standalone.sch (EAGLE design)
At the start: 64 parts, among them IC1 LMC6484P, IC2 LM555N, IC3 74HCT74N, IC4 4044N, IC8 7805TV, T1 2N2222, T2 2N2222, U1 MAX4544, U4 MotA

Commit message: Finished routing traces, all DRC okay
Parts:
- added J1: J5MM, jumper:J5MM
Connections:
- removed net N$30 (its old number): 16X2.8, U3.6
- new net N$20: 16X2.10, U3.2
- new net N$31: 16X2.6, U3.6
- net +5V: now also J1.1
- net N$24: now also 16X2.9, U3.3; no longer 16X2.10, U3.8
- net N$29: now also 16X2.8, U3.4; no longer 16X2.9, U3.7
- net N$32: now also 16X2.5, U3.7; no longer 16X2.6, U3.4
- net N$41: now also 16X2.4, U3.8; no longer 16X2.5, U3.3
- net N$46: now also J1.2, U3.5V; no longer 16X2.4, U3.2
Changed lines of the file:
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@@
 <grid distance="0.1" unitdist="inch" unit="inch" style="lines" multiple="1" display="no" altdistance="0.01" altunitdist="inch" altunit="inch"/>
 <layers>
-<layer number="1" name="Top" color="4" fill="1" visible="yes" active="no"/>
-<layer number="16" name="Bottom" color="1" fill="1" visible="yes" active="no"/>
-<layer number="17" name="Pads" color="2" fill="1" visible="yes" active="no"/>
-<layer number="18" name="Vias" color="2" fill="1" visible="yes" active="no"/>
-<layer number="19" name="Unrouted" color="6" fill="1" visible="yes" active="no"/>
-<layer number="20" name="Dimension" color="15" fill="1" visible="yes" active="no"/>
-<layer number="21" name="tPlace" color="7" fill="1" visible="yes" active="no"/>
-<layer number="22" name="bPlace" color="7" fill="1" visible="yes" active="no"/>
-<layer number="23" name="tOrigins" color="15" fill="1" visible="yes" active="no"/>
-<layer number="24" name="bOrigins" color="15" fill="1" visible="yes" active="no"/>
-<layer number="25" name="tNames" color="7" fill="1" visible="yes" active="no"/>
-<layer number="26" name="bNames" color="7" fill="1" visible="yes" active="no"/>
-<layer number="27" name="tValues" color="7" fill="1" visible="yes" active="no"/>
-<layer number="28" name="bValues" color="7" fill="1" visible="yes" active="no"/>
+<layer number="1" name="Top" color="4" fill="1" visible="no" active="no"/>
+<layer number="16" name="Bottom" color="1" fill="1" visible="no" active="no"/>
+<layer number="17" name="Pads" color="2" fill="1" visible="no" active="no"/>
+<layer number="18" name="Vias" color="2" fill="1" visible="no" active="no"/>
+<layer number="19" name="Unrouted" color="6" fill="1" visible="no" active="no"/>
+<layer number="20" name="Dimension" color="15" fill="1" visible="no" active="no"/>
+<layer number="21" name="tPlace" color="7" fill="1" visible="no" active="no"/>
+<layer number="22" name="bPlace" color="7" fill="1" visible="no" active="no"/>
+<layer number="23" name="tOrigins" color="15" fill="1" visible="no" active="no"/>
+<layer number="24" name="bOrigins" color="15" fill="1" visible="no" active="no"/>
+<layer number="25" name="tNames" color="7" fill="1" visible="no" active="no"/>
+<layer number="26" name="bNames" color="7" fill="1" visible="no" active="no"/>
+<layer number="27" name="tValues" color="7" fill="1" visible="no" active="no"/>
+<layer number="28" name="bValues" color="7" fill="1" visible="no" active="no"/>
 <layer number="29" name="tStop" color="7" fill="3" visible="no" active="no"/>
 <layer number="30" name="bStop" color="7" fill="6" visible="no" active="no"/>
@@
 <layer number="35" name="tGlue" color="7" fill="4" visible="no" active="no"/>
 <layer number="36" name="bGlue" color="7" fill="5" visible="no" active="no"/>
-<layer number="37" name="tTest" color="7" fill="1" visible="yes" active="no"/>
-<layer number="38" name="bTest" color="7" fill="1" visible="yes" active="no"/>
+<layer number="37" name="tTest" color="7" fill="1" visible="no" active="no"/>
+<layer number="38" name="bTest" color="7" fill="1" visible="no" active="no"/>
 <layer number="39" name="tKeepout" color="4" fill="11" visible="no" active="no"/>
 <layer number="40" name="bKeepout" color="1" fill="11" visible="no" active="no"/>
@@
 <layer number="44" name="Drills" color="7" fill="1" visible="no" active="no"/>
 <layer number="45" name="Holes" color="7" fill="1" visible="no" active="no"/>
-<layer number="46" name="Milling" color="3" fill="1" visible="yes" active="no"/>
-<layer number="47" name="Measures" color="7" fill="1" visible="yes" active="no"/>
-<layer number="48" name="Document" color="7" fill="1" visible="yes" active="no"/>
-<layer number="49" name="Reference" color="7" fill="1" visible="yes" active="no"/>
-<layer number="50" name="dxf" color="7" fill="1" visible="yes" active="no"/>
-<layer number="51" name="tDocu" color="7" fill="1" visible="yes" active="no"/>
-<layer number="52" name="bDocu" color="7" fill="1" visible="yes" active="no"/>
-<layer number="53" name="tGND_GNDA" color="7" fill="9" visible="yes" active="no"/>
-<layer number="54" name="bGND_GNDA" color="1" fill="9" visible="yes" active="no"/>
-<layer number="56" name="wert" color="7" fill="1" visible="yes" active="no"/>
-<layer number="57" name="tCAD" color="7" fill="1" visible="yes" active="no"/>
+<layer number="46" name="Milling" color="3" fill="1" visible="no" active="no"/>
+<layer number="47" name="Measures" color="7" fill="1" visible="no" active="no"/>
+<layer number="48" name="Document" color="7" fill="1" visible="no" active="no"/>
+<layer number="49" name="Reference" color="7" fill="1" visible="no" active="no"/>
+<layer number="50" name="dxf" color="7" fill="1" visible="no" active="no"/>
+<layer number="51" name="tDocu" color="7" fill="1" visible="no" active="no"/>
+<layer number="52" name="bDocu" color="7" fill="1" visible="no" active="no"/>
+<layer number="53" name="tGND_GNDA" color="7" fill="9" visible="no" active="no"/>
+<layer number="54" name="bGND_GNDA" color="1" fill="9" visible="no" active="no"/>
+<layer number="56" name="wert" color="7" fill="1" visible="no" active="no"/>
+<layer number="57" name="tCAD" color="7" fill="1" visible="no" active="no"/>
 <layer number="90" name="Modules" color="5" fill="1" visible="yes" active="yes"/>
 <layer number="91" name="Nets" color="2" fill="1" visible="yes" active="yes"/>
@@
 <part name="JP2" library="pinhead" deviceset="PINHD-1X2" device=""/>
 <part name="SUPPLY31" library="supply2" deviceset="+5V" device=""/>
+<part name="J1" library="jumper" deviceset="J" device="5MM"/>
+<part name="SUPPLY32" library="supply2" deviceset="+5V" device=""/>
 </parts>
 <sheets>
@@
 <instance part="IC3" gate="B" x="25.4" y="129.54"/>
 <instance part="SUPPLY31" gate="+5V" x="10.16" y="139.7"/>
+<instance part="J1" gate="1" x="213.36" y="45.72"/>
+<instance part="SUPPLY32" gate="+5V" x="203.2" y="50.8"/>
 </instances>
 <busses>
@@
 <wire x1="12.7" y1="127" x2="10.16" y2="127" width="0.1524" layer="91"/>
 <junction x="10.16" y="127"/>
+</segment>
+<segment>
+<pinref part="SUPPLY32" gate="+5V" pin="+5V"/>
+<wire x1="203.2" y1="48.26" x2="203.2" y2="45.72" width="0.1524" layer="91"/>
+<pinref part="J1" gate="1" pin="1"/>
+<wire x1="203.2" y1="45.72" x2="208.28" y2="45.72" width="0.1524" layer="91"/>
 </segment>
 </net>
@@
 </segment>
 </net>
+<net name="N$20" class="0">
+<segment>
+<pinref part="16X2" gate="G$1" pin="10"/>
+<wire x1="259.08" y1="73.66" x2="259.08" y2="43.18" width="0.1524" layer="91"/>
+<pinref part="U3" gate="G$1" pin="2"/>
+<wire x1="259.08" y1="43.18" x2="246.38" y2="43.18" width="0.1524" layer="91"/>
+</segment>
+</net>
 <net name="N$24" class="0">
 <segment>
-<pinref part="U3" gate="G$1" pin="8"/>
-<pinref part="16X2" gate="G$1" pin="10"/>
-<wire x1="246.38" y1="27.94" x2="259.08" y2="27.94" width="0.1524" layer="91"/>
-<wire x1="259.08" y1="27.94" x2="259.08" y2="73.66" width="0.1524" layer="91"/>
+<pinref part="U3" gate="G$1" pin="3"/>
+<pinref part="16X2" gate="G$1" pin="9"/>
+<wire x1="246.38" y1="40.64" x2="261.62" y2="40.64" width="0.1524" layer="91"/>
+<wire x1="261.62" y1="40.64" x2="261.62" y2="73.66" width="0.1524" layer="91"/>
 </segment>
 </net>
 <net name="N$29" class="0">
 <segment>
-<pinref part="16X2" gate="G$1" pin="9"/>
-<wire x1="261.62" y1="73.66" x2="261.62" y2="30.48" width="0.1524" layer="91"/>
-<pinref part="U3" gate="G$1" pin="7"/>
-<wire x1="261.62" y1="30.48" x2="246.38" y2="30.48" width="0.1524" layer="91"/>
+<pinref part="U3" gate="G$1" pin="4"/>
+<pinref part="16X2" gate="G$1" pin="8"/>
+<wire x1="246.38" y1="38.1" x2="264.16" y2="38.1" width="0.1524" layer="91"/>
+<wire x1="264.16" y1="38.1" x2="264.16" y2="73.66" width="0.1524" layer="91"/>
 </segment>
 </net>
 <net name="N$30" class="0">
-<segment>
-<pinref part="U3" gate="G$1" pin="6"/>
-<wire x1="246.38" y1="33.02" x2="264.16" y2="33.02" width="0.1524" layer="91"/>
-<pinref part="16X2" gate="G$1" pin="8"/>
-<wire x1="264.16" y1="33.02" x2="264.16" y2="73.66" width="0.1524" layer="91"/>
-</segment>
-</net>
-<net name="N$31" class="0">
 <segment>
 <pinref part="U3" gate="G$1" pin="5"/>
@@
 </segment>
 </net>
+<net name="N$31" class="0">
+<segment>
+<pinref part="U3" gate="G$1" pin="6"/>
+<pinref part="16X2" gate="G$1" pin="6"/>
+<wire x1="246.38" y1="33.02" x2="269.24" y2="33.02" width="0.1524" layer="91"/>
+<wire x1="269.24" y1="33.02" x2="269.24" y2="73.66" width="0.1524" layer="91"/>
+</segment>
+</net>
 <net name="N$32" class="0">
 <segment>
-<pinref part="U3" gate="G$1" pin="4"/>
-<wire x1="246.38" y1="38.1" x2="269.24" y2="38.1" width="0.1524" layer="91"/>
-<wire x1="269.24" y1="38.1" x2="269.24" y2="73.66" width="0.1524" layer="91"/>
-<pinref part="16X2" gate="G$1" pin="6"/>
+<pinref part="U3" gate="G$1" pin="7"/>
+<pinref part="16X2" gate="G$1" pin="5"/>
+<wire x1="246.38" y1="30.48" x2="271.78" y2="30.48" width="0.1524" layer="91"/>
+<wire x1="271.78" y1="30.48" x2="271.78" y2="73.66" width="0.1524" layer="91"/>
 </segment>
 </net>
 <net name="N$41" class="0">
 <segment>
-<pinref part="U3" gate="G$1" pin="3"/>
-<pinref part="16X2" gate="G$1" pin="5"/>
-<wire x1="246.38" y1="40.64" x2="271.78" y2="40.64" width="0.1524" layer="91"/>
-<wire x1="271.78" y1="40.64" x2="271.78" y2="73.66" width="0.1524" layer="91"/>
+<pinref part="U3" gate="G$1" pin="8"/>
+<pinref part="16X2" gate="G$1" pin="4"/>
+<wire x1="246.38" y1="27.94" x2="274.32" y2="27.94" width="0.1524" layer="91"/>
+<wire x1="274.32" y1="27.94" x2="274.32" y2="73.66" width="0.1524" layer="91"/>
 </segment>
 </net>
 <net name="N$46" class="0">
 <segment>
-<pinref part="U3" gate="G$1" pin="2"/>
-<pinref part="16X2" gate="G$1" pin="4"/>
-<wire x1="246.38" y1="43.18" x2="274.32" y2="43.18" width="0.1524" layer="91"/>
-<wire x1="274.32" y1="43.18" x2="274.32" y2="73.66" width="0.1524" layer="91"/>
-</segment>
-</net>
+<pinref part="U3" gate="G$1" pin="5V"/>
+<pinref part="J1" gate="1" pin="2"/>
+<wire x1="220.98" y1="45.72" x2="218.44" y2="45.72" width="0.1524" layer="91"/>
+</segment>
+</net>
