File: nephelometer/circuitry/band-psd-micro-standalone.sch (EAGLE design)
At the start: 65 parts, among them IC1 LMC6484P, IC2 LM555N, IC3 74HCT74N, IC4 4044N, IC8 7805TV, J1 J5MM, T1 2N2222, T2 2N2222, U1 MAX4544, U4 MotA

Commit message: Finished placement labels and added test point
Parts:
- added TP1: (no value), ingolia:TEST_POINT
Connections:
- net 2.5V: now also TP1.+
- net N$28: now also TP1.-
Changed lines of the file:
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@@
 <part name="J1" library="jumper" deviceset="J" device="5MM"/>
 <part name="SUPPLY32" library="supply2" deviceset="+5V" device=""/>
+<part name="TP1" library="ingolia" deviceset="TEST_POINT" device=""/>
 </parts>
 <sheets>
@@
 <instance part="J1" gate="1" x="213.36" y="45.72"/>
 <instance part="SUPPLY32" gate="+5V" x="203.2" y="50.8"/>
+<instance part="TP1" gate="G$1" x="215.9" y="22.86"/>
 </instances>
 <busses>
@@
 <segment>
 <pinref part="IC5" gate="G$1" pin="IN+"/>
-<wire x1="210.82" y1="-2.54" x2="210.82" y2="5.08" width="0.1524" layer="91"/>
 <label x="210.82" y="0" size="1.778" layer="95" rot="R90"/>
+<pinref part="TP1" gate="G$1" pin="+"/>
+<wire x1="213.36" y1="25.4" x2="210.82" y2="25.4" width="0.1524" layer="91"/>
+<wire x1="210.82" y1="25.4" x2="210.82" y2="-2.54" width="0.1524" layer="91"/>
 </segment>
 </net>
@@
 <junction x="203.2" y="33.02"/>
 <pinref part="IC5" gate="G$1" pin="IN-"/>
-<wire x1="208.28" y1="33.02" x2="208.28" y2="-2.54" width="0.1524" layer="91"/>
-</segment>
-</net>
+<wire x1="208.28" y1="33.02" x2="208.28" y2="22.86" width="0.1524" layer="91"/>
+<pinref part="TP1" gate="G$1" pin="-"/>
+<wire x1="208.28" y1="22.86" x2="208.28" y2="-2.54" width="0.1524" layer="91"/>
+<wire x1="213.36" y1="22.86" x2="208.28" y2="22.86" width="0.1524" layer="91"/>
+<junction x="208.28" y="22.86"/>
+</segment>
+</net>

Commit message: Finished BOM part assignments
Parts:
- C10, C11, C16, C8: DIGIKEY# (none) -> BC1084CT-ND
- C9: DIGIKEY# (none) -> 445-8384-ND; MANF (none) -> TDK Corporation; MANF# (none) -> FK18C0G1H103J
- IC1: DIGIKEY2# (none) -> AE10012-ND
- IC2: DIGIKEY# (none) -> LM555CNFS-ND; DIGIKEY2# (none) -> AE9986-ND; MANF (none) -> Fairchild Semiconductor; MANF# (none) -> LM555CN
- IC3: DIGIKEY# (none) -> 296-1625-5-ND; DIGIKEY2# (none) -> AE10012-ND; MANF (none) -> Texas Instruments; MANF# (none) -> SN74HCT74N
- IC4: DIGIKEY# (none) -> 296-2051-5-ND; DIGIKEY2# (none) -> AE9992-ND; MANF (none) -> Texas Instruments; MANF# (none) -> CD4044BE
- IC5, U1: DIGIKEY2# (none) -> AE9986-ND
- JP1: DIGIKEY# (none) -> 475-3002-ND; DIGIKEY2# (none) -> 492-1502-ND; MANF (none) -> OSRAM Opto Semiconductors Inc; MANF# (none) -> SFH 4547; MANF2 (none) -> Bivar Inc; MANF2# (none) -> CR-174
- LED1: DIGIKEY# (none) -> 160-1139-ND; MANF (none) -> Lite-On Inc; MANF# (none) -> LTL-4221N
- Q1: DIGIKEY# (none) -> 160-1030-ND; MANF (none) -> Lite-On Inc; MANF# (none) -> LTR-4206E
- Q2: DIGIKEY# (none) -> IRLB8721PBF-ND
- R10, R11, R13: DIGIKEY# (none) -> S4.7KQCT-ND; MANF (none) -> Stackpole Electronics Inc; MANF# (none) -> CFM14JT4K70
- R15: value 6.3R -> 6.2R; DIGIKEY# (none) -> PPC6.2W-1CT-ND; MANF (none) -> Vishay BC Components; MANF# (none) -> PR01000106208JR500
- R16: DIGIKEY# (none) -> CF14JT330RCT-ND; MANF (none) -> Stackpole Electronics Inc; MANF# (none) -> CF14JT330R
- R8, R9: DIGIKEY# (none) -> S4.7KCACT-ND; MANF (none) -> Stackpole Electronics Inc; MANF# (none) -> RNMF14FTC4K70
- RN1: DIGIKEY# (none) -> 4609X-101-103LF-ND; MANF (none) -> Bourns Inc.; MANF# (none) -> 4609X-101-103LF
- T1, T2: DIGIKEY# (none) -> PN2222ATFCT-ND; MANF (none) -> Fairchild Semiconductor; MANF# (none) -> PN2222ATF
- TM1: DIGIKEY# (none) -> 3386P-103LF-ND; MANF (none) -> Bourns Inc.; MANF# (none) -> 3386P-1-103LF
- U$5, U$6, U$8: DIGIKEY# (none) -> 563-1183-ND
- U$9: DIGIKEY# (none) -> 563-1183-ND; MANF (none) -> Copal Electronics Inc; MANF# (none) -> APE1F-5M-10-Z
- U2: DIGIKEY# (none) -> CP-5-ND; MANF (none) -> CUI Inc; MANF# (none) -> PJ-005A
- U4: DIGIKEY# (none) -> SC1455-ND; MANF (none) -> Switchcraft Inc.; MANF# (none) -> 35PM1

Commit message: Finished BOM attributes needed for 15-02-01 test fabrication
Parts:
- J1: DIGIKEY# (none) -> 0.0EBK-ND; MANF (none) -> Yageo; MANF# (none) -> ZOR-12-B-52-0R
- U3: DIGIKEY# (none) -> 1050-1066-ND; DIGIKEY2# (none) -> S7050-ND x 2; MANF (none) -> Arduino; MANF# (none) -> A000053; MANF2 (none) -> Sullins Connector Solutions; MANF2# (none) -> PPPC171LFBN-RC
Changed lines of the file:
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@@
 <grid distance="0.1" unitdist="inch" unit="inch" style="lines" multiple="1" display="no" altdistance="0.01" altunitdist="inch" altunit="inch"/>
 <layers>
-<layer number="1" name="Top" color="4" fill="1" visible="yes" active="no"/>
-<layer number="16" name="Bottom" color="1" fill="1" visible="yes" active="no"/>
-<layer number="17" name="Pads" color="2" fill="1" visible="yes" active="no"/>
-<layer number="18" name="Vias" color="2" fill="1" visible="yes" active="no"/>
-<layer number="19" name="Unrouted" color="6" fill="1" visible="yes" active="no"/>
-<layer number="20" name="Dimension" color="15" fill="1" visible="yes" active="no"/>
-<layer number="21" name="tPlace" color="7" fill="1" visible="yes" active="no"/>
-<layer number="22" name="bPlace" color="7" fill="1" visible="yes" active="no"/>
-<layer number="23" name="tOrigins" color="15" fill="1" visible="yes" active="no"/>
-<layer number="24" name="bOrigins" color="15" fill="1" visible="yes" active="no"/>
-<layer number="25" name="tNames" color="7" fill="1" visible="yes" active="no"/>
-<layer number="26" name="bNames" color="7" fill="1" visible="yes" active="no"/>
-<layer number="27" name="tValues" color="7" fill="1" visible="yes" active="no"/>
-<layer number="28" name="bValues" color="7" fill="1" visible="yes" active="no"/>
+<layer number="1" name="Top" color="4" fill="1" visible="no" active="no"/>
+<layer number="16" name="Bottom" color="1" fill="1" visible="no" active="no"/>
+<layer number="17" name="Pads" color="2" fill="1" visible="no" active="no"/>
+<layer number="18" name="Vias" color="2" fill="1" visible="no" active="no"/>
+<layer number="19" name="Unrouted" color="6" fill="1" visible="no" active="no"/>
+<layer number="20" name="Dimension" color="15" fill="1" visible="no" active="no"/>
+<layer number="21" name="tPlace" color="7" fill="1" visible="no" active="no"/>
+<layer number="22" name="bPlace" color="7" fill="1" visible="no" active="no"/>
+<layer number="23" name="tOrigins" color="15" fill="1" visible="no" active="no"/>
+<layer number="24" name="bOrigins" color="15" fill="1" visible="no" active="no"/>
+<layer number="25" name="tNames" color="7" fill="1" visible="no" active="no"/>
+<layer number="26" name="bNames" color="7" fill="1" visible="no" active="no"/>
+<layer number="27" name="tValues" color="7" fill="1" visible="no" active="no"/>
+<layer number="28" name="bValues" color="7" fill="1" visible="no" active="no"/>
 <layer number="29" name="tStop" color="7" fill="3" visible="no" active="no"/>
 <layer number="30" name="bStop" color="7" fill="6" visible="no" active="no"/>
@@
 <layer number="35" name="tGlue" color="7" fill="4" visible="no" active="no"/>
 <layer number="36" name="bGlue" color="7" fill="5" visible="no" active="no"/>
-<layer number="37" name="tTest" color="7" fill="1" visible="yes" active="no"/>
-<layer number="38" name="bTest" color="7" fill="1" visible="yes" active="no"/>
+<layer number="37" name="tTest" color="7" fill="1" visible="no" active="no"/>
+<layer number="38" name="bTest" color="7" fill="1" visible="no" active="no"/>
 <layer number="39" name="tKeepout" color="4" fill="11" visible="no" active="no"/>
 <layer number="40" name="bKeepout" color="1" fill="11" visible="no" active="no"/>
@@
 <layer number="44" name="Drills" color="7" fill="1" visible="no" active="no"/>
 <layer number="45" name="Holes" color="7" fill="1" visible="no" active="no"/>
-<layer number="46" name="Milling" color="3" fill="1" visible="yes" active="no"/>
-<layer number="47" name="Measures" color="7" fill="1" visible="yes" active="no"/>
-<layer number="48" name="Document" color="7" fill="1" visible="yes" active="no"/>
-<layer number="49" name="Reference" color="7" fill="1" visible="yes" active="no"/>
-<layer number="50" name="dxf" color="7" fill="1" visible="yes" active="no"/>
-<layer number="51" name="tDocu" color="7" fill="1" visible="yes" active="no"/>
-<layer number="52" name="bDocu" color="7" fill="1" visible="yes" active="no"/>
-<layer number="53" name="tGND_GNDA" color="7" fill="9" visible="yes" active="no"/>
-<layer number="54" name="bGND_GNDA" color="1" fill="9" visible="yes" active="no"/>
-<layer number="56" name="wert" color="7" fill="1" visible="yes" active="no"/>
-<layer number="57" name="tCAD" color="7" fill="1" visible="yes" active="no"/>
+<layer number="46" name="Milling" color="3" fill="1" visible="no" active="no"/>
+<layer number="47" name="Measures" color="7" fill="1" visible="no" active="no"/>
+<layer number="48" name="Document" color="7" fill="1" visible="no" active="no"/>
+<layer number="49" name="Reference" color="7" fill="1" visible="no" active="no"/>
+<layer number="50" name="dxf" color="7" fill="1" visible="no" active="no"/>
+<layer number="51" name="tDocu" color="7" fill="1" visible="no" active="no"/>
+<layer number="52" name="bDocu" color="7" fill="1" visible="no" active="no"/>
+<layer number="53" name="tGND_GNDA" color="7" fill="9" visible="no" active="no"/>
+<layer number="54" name="bGND_GNDA" color="1" fill="9" visible="no" active="no"/>
+<layer number="56" name="wert" color="7" fill="1" visible="no" active="no"/>
+<layer number="57" name="tCAD" color="7" fill="1" visible="no" active="no"/>
 <layer number="90" name="Modules" color="5" fill="1" visible="yes" active="yes"/>
 <layer number="91" name="Nets" color="2" fill="1" visible="yes" active="yes"/>
@@
 <attribute name="MANF#" value="FK16C0G1H473J"/>
 </part>
-<part name="U3" library="adafruit" deviceset="ARDUINOMICRO" device=""/>
+<part name="U3" library="adafruit" deviceset="ARDUINOMICRO" device="">
+<attribute name="DIGIKEY#" value="1050-1066-ND"/>
+<attribute name="DIGIKEY2#" value="S7050-ND x 2"/>
+<attribute name="MANF" value="Arduino"/>
+<attribute name="MANF#" value="A000053"/>
+<attribute name="MANF2" value="Sullins Connector Solutions"/>
+<attribute name="MANF2#" value="PPPC171LFBN-RC"/>
+</part>
 <part name="U2" library="ingolia" deviceset="DC-IN-PANEL-NODETECT" device="">
 <attribute name="DIGIKEY#" value="CP-5-ND"/>
@@
 <part name="JP2" library="pinhead" deviceset="PINHD-1X2" device=""/>
 <part name="SUPPLY31" library="supply2" deviceset="+5V" device=""/>
-<part name="J1" library="jumper" deviceset="J" device="5MM"/>
+<part name="J1" library="jumper" deviceset="J" device="5MM">
+<attribute name="DIGIKEY#" value="0.0EBK-ND"/>
+<attribute name="MANF" value="Yageo"/>
+<attribute name="MANF#" value="ZOR-12-B-52-0R"/>
+</part>
 <part name="SUPPLY32" library="supply2" deviceset="+5V" device=""/>
 <part name="TP1" library="ingolia" deviceset="TEST_POINT" device=""/>
@@
 <attribute name="MANF#" x="180.34" y="43.18" size="1.778" layer="96" rot="R90" display="off"/>
 </instance>
-<instance part="U3" gate="G$1" x="233.68" y="38.1" rot="MR90"/>
+<instance part="U3" gate="G$1" x="233.68" y="38.1" rot="MR90">
+<attribute name="DIGIKEY#" x="233.68" y="38.1" size="1.778" layer="96" rot="MR90" display="off"/>
+<attribute name="MANF" x="233.68" y="38.1" size="1.778" layer="96" rot="MR90" display="off"/>
+<attribute name="MANF#" x="233.68" y="38.1" size="1.778" layer="96" rot="MR90" display="off"/>
+<attribute name="DIGIKEY2#" x="233.68" y="38.1" size="1.778" layer="96" rot="MR90" display="off"/>
+<attribute name="MANF2" x="233.68" y="38.1" size="1.778" layer="96" rot="MR90" display="off"/>
+<attribute name="MANF2#" x="233.68" y="38.1" size="1.778" layer="96" rot="MR90" display="off"/>
+</instance>
 <instance part="U2" gate="G$1" x="175.26" y="119.38">
 <attribute name="DIGIKEY#" x="175.26" y="119.38" size="1.778" layer="96" display="off"/>
@@
 <instance part="IC3" gate="B" x="25.4" y="129.54"/>
 <instance part="SUPPLY31" gate="+5V" x="10.16" y="139.7"/>
-<instance part="J1" gate="1" x="213.36" y="45.72"/>
+<instance part="J1" gate="1" x="213.36" y="45.72">
+<attribute name="DIGIKEY#" x="213.36" y="45.72" size="1.778" layer="96" display="off"/>
+<attribute name="MANF" x="213.36" y="45.72" size="1.778" layer="96" display="off"/>
+<attribute name="MANF#" x="213.36" y="45.72" size="1.778" layer="96" display="off"/>
+</instance>
 <instance part="SUPPLY32" gate="+5V" x="203.2" y="50.8"/>
 <instance part="TP1" gate="G$1" x="215.9" y="22.86"/>

Commit message: Fixup extraneous space in part #
Parts:
- R8: DIGIKEY# S4.7KCACT-ND -> S4.7KCACT-ND
Changed lines of the file:
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@@
 </part>
 <part name="R8" library="adafruit" deviceset="R-US_" device="0204/2V" value="4K7">
-<attribute name="DIGIKEY#" value="S4.7KCACT-ND "/>
+<attribute name="DIGIKEY#" value="S4.7KCACT-ND"/>
 <attribute name="MANF" value="Stackpole Electronics Inc"/>
 <attribute name="MANF#" value="RNMF14FTC4K70"/>
