File: nephelometer/circuitry/band-dsp-micro.sch (EAGLE design)
At the start: 36 parts, among them IC8 7805TV, J1 J5MM, T1 2N2222, T2 2N2222, U4 MotA

Commit message: Finalized minimal turbidostat circuit with Arduino Micro control
Parts:
- removed C16: 100n, adafruit:C-US025-025X050
- removed IC6: (no value), v-reg:LM317L
- removed R11, R13: 4K7, adafruit:R-US_0204/2V
- removed R15: 6.2R, adafruit:R-US_0204/2V
- removed U4: MotA, ingolia:1X02_MOTOR
- added C6: 100n, adafruit:C-US025-025X050
- added R6: 2M0, adafruit:R-US_0309/V
- added R7, R8: 4K7, adafruit:R-US_0204/2V
- added U1: (no value), ingolia:LMC6482
- C1: value 2.2nF -> 100nF; device adafruit:C-US025-024X044 -> adafruit:C-US025-025X050; DIGIKEY# BC1029CT-ND -> BC1084CT-ND; MANF# K222J15C0GF5TL2 -> K104K15X7RF5TL2
- C2: value 100nF -> 2.2nF; device adafruit:C-US025-025X050 -> adafruit:C-US025-024X044; DIGIKEY# BC1084CT-ND -> BC1029CT-ND; MANF# K104K15X7RF5TL2 -> K222J15C0GF5TL2
- IC1: device ingolia:LMC6482 -> v-reg:LM317L; DIGIKEY# LMC6484AIN/NOPB-ND -> 296-33312-5-ND; DIGIKEY2# AE10012-ND -> (none); MANF# LMC6484AIN/NOPB -> LM317LCLP
- J1: value J5MM -> 2.1MMJACKTHM; device jumper:J5MM -> adafruit:2.1MMJACKTHM; DIGIKEY# 0.0EBK-ND -> CP-102A-ND; MANF Yageo -> CUI Inc; MANF# ZOR-12-B-52-0R -> PJ-102A
- R2: value 1K0 -> 120; device adafruit:R-US_0204/5 -> adafruit:R-US_0204/2V; DIGIKEY# S1KCACT-ND -> S120CACT-ND; MANF# RNMF14FTC1K00 -> RNMF14FTC120R
- R4: value 120 -> 10K; device adafruit:R-US_0204/2V -> adafruit:R-US_0204/5; DIGIKEY# S120CACT-ND -> S10KCACT-ND; MANF# RNMF14FTC120R -> RNMF14FTC10K0
- R5: value 330K -> 10R; device adafruit:R-US_0309/V -> adafruit:R-US_0204/2V; DIGIKEY# RNV14FAL330KCT-ND -> PPC10W-1CT-ND; MANF Stackpole Electronics Inc -> Vishay BC Components; MANF# RNV14FAL330K -> PR01000101009JR500
- U2: value (none) -> MotA; device ingolia:DC-IN-PANEL-NODETECT -> ingolia:1X02_MOTOR; DIGIKEY# CP-5-ND -> SC1455-ND; MANF CUI Inc -> Switchcraft Inc.; MANF# PJ-005A -> 35PM1
- renumbered C14 to C7, C17 to C8, C18 to C9, C19 to C10, IC5 to IC2, IC8 to IC3, R16 to R9
Connections:
- removed net CS_ADC: IC2.SHDN, U3.2
- removed net N$46: J1.2, U3.5V
- new net N$7: IC2.SHDN, U3.A5
- net +12V: now also J1.TIP, Q4.G, R7.2, U2.+; no longer Q3.G, R13.2, U2.PWR, U4.+
- net +5V: now also C1.2, C6.1, IC1.IN, U1P.V+, U3.5V; no longer C16.1, C2.2, IC1P.V+, IC6.IN, J1.1
- net 2.5V: now also IC1.OUT, R2.1, U1A.+IN, U1B.+IN; no longer IC1A.+IN, IC1B.+IN, IC6.OUT, R3.1
- net GND: now also C1.1, C6.2, Q3.S, Q4.D, R3.1, R5.1, U1P.V-; no longer C16.2, C2.1, IC1P.V-, Q3.D, Q4.S, R15.1, R4.1
- net LEDCTRL: now also R8.2, T2.B; no longer R11.2, T1.B
- net N$1: now also C2.1, U1B.-IN; no longer C1.1, IC1B.-IN
- net N$14: now also R5.2, T1.B; no longer R15.2, T2.B
- net N$19: now also Q3.G; no longer Q4.G
- net N$2: now also R4.1; no longer R2.1
- net N$22: now also C2.2, U1B.OUT; no longer C1.2, IC1B.OUT
- net N$25: now also R4.2, R6.1, U1A.-IN; no longer IC1A.-IN, R2.2, R5.1
- net N$26: now also R6.2, U1A.OUT; no longer IC1A.OUT, R5.2
- net N$3: now also Q3.D, U2.-; no longer Q4.D, U4.-
- net N$35: now also IC1.ADJ, R2.2; no longer IC6.ADJ, R4.2
- net N$47: now also J1.RING, Q4.S; no longer Q3.S, U2.GND
- net N$5: now also R8.1, U3.A0; no longer R11.1, U3.12
- net N$8: now also R7.1; no longer R13.1
Other:
- moved on the sheet: C1, C2, C4, JP1, Q1, Q2, Q3, Q4, R1, R2, R3, R4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

Commit message: Updated parts list based on first round of building turbidostats
Parts:
- J1: DIGIKEY2# (none) -> T1071-P5P-ND; MANF2 (none) -> CUI Inc; MANF2# (none) -> EPSA120200U-P5P-SZ
- U1: DIGIKEY# LMC6484AIN/NOPB-ND -> LMC6482AIN/NOPB-ND; DIGIKEY2# AE10012-ND -> AE9986-ND; MANF# LMC6484AIN/NOPB -> LMC6482AIN/NOPB
- U3: DIGIKEY2# S7050-ND x 2 -> S7050-ND; DIGIKEY3# (none) -> S7050-ND; DIGIKEY4# (none) -> AE10419-ND; MANF3 (none) -> Sullins Connector Solutions; MANF3# (none) -> PPPC171LFBN-RC; MANF4 (none) -> Assmann WSW Components; MANF4# (none) -> AK67421-1
Changed lines of the file:
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@@
 <part name="SUPPLY3" library="supply2" deviceset="GND" device=""/>
 <part name="U1" library="ingolia" deviceset="LMC6482" device="">
-<attribute name="DIGIKEY#" value="LMC6484AIN/NOPB-ND"/>
-<attribute name="DIGIKEY2#" value="AE10012-ND"/>
+<attribute name="DIGIKEY#" value="LMC6482AIN/NOPB-ND"/>
+<attribute name="DIGIKEY2#" value="AE9986-ND"/>
 <attribute name="MANF" value="Texas Instruments"/>
-<attribute name="MANF#" value="LMC6484AIN/NOPB"/>
+<attribute name="MANF#" value="LMC6482AIN/NOPB"/>
 </part>
 <part name="R4" library="adafruit" deviceset="R-US_" device="0204/5" value="10K">
@@
 <part name="U3" library="adafruit" deviceset="ARDUINOMICRO" device="">
 <attribute name="DIGIKEY#" value="1050-1066-ND"/>
-<attribute name="DIGIKEY2#" value="S7050-ND x 2"/>
+<attribute name="DIGIKEY2#" value="S7050-ND"/>
+<attribute name="DIGIKEY3#" value="S7050-ND"/>
+<attribute name="DIGIKEY4#" value="AE10419-ND"/>
 <attribute name="MANF" value="Arduino"/>
 <attribute name="MANF#" value="A000053"/>
 <attribute name="MANF2" value="Sullins Connector Solutions"/>
 <attribute name="MANF2#" value="PPPC171LFBN-RC"/>
+<attribute name="MANF3" value="Sullins Connector Solutions"/>
+<attribute name="MANF3#" value="PPPC171LFBN-RC"/>
+<attribute name="MANF4" value="Assmann WSW Components"/>
+<attribute name="MANF4#" value="AK67421-1"/>
 </part>
 <part name="Q4" library="ingolia" deviceset="IRLB8721" device="">
@@
 <part name="J1" library="adafruit" deviceset="2.1MMJACK" device="THM">
 <attribute name="DIGIKEY#" value="CP-102A-ND "/>
+<attribute name="DIGIKEY2#" value="T1071-P5P-ND "/>
 <attribute name="MANF" value="CUI Inc"/>
 <attribute name="MANF#" value="PJ-102A"/>
+<attribute name="MANF2" value="CUI Inc"/>
+<attribute name="MANF2#" value="EPSA120200U-P5P-SZ"/>
 </part>
 </parts>
@@
 <attribute name="MANF2" x="233.68" y="38.1" size="1.778" layer="96" rot="MR90" display="off"/>
 <attribute name="MANF2#" x="233.68" y="38.1" size="1.778" layer="96" rot="MR90" display="off"/>
+<attribute name="DIGIKEY3#" x="233.68" y="38.1" size="1.778" layer="96" rot="MR90" display="off"/>
+<attribute name="MANF3" x="233.68" y="38.1" size="1.778" layer="96" rot="MR90" display="off"/>
+<attribute name="MANF3#" x="233.68" y="38.1" size="1.778" layer="96" rot="MR90" display="off"/>
+<attribute name="DIGIKEY4#" x="233.68" y="38.1" size="1.778" layer="96" rot="MR90" display="off"/>
+<attribute name="MANF4" x="233.68" y="38.1" size="1.778" layer="96" rot="MR90" display="off"/>
+<attribute name="MANF4#" x="233.68" y="38.1" size="1.778" layer="96" rot="MR90" display="off"/>
 </instance>
 <instance part="Q4" gate="G$1" x="205.74" y="81.28" rot="R270">
@@
 <attribute name="MANF" x="193.04" y="88.9" size="1.778" layer="96" display="off"/>
 <attribute name="MANF#" x="193.04" y="88.9" size="1.778" layer="96" display="off"/>
+<attribute name="DIGIKEY2#" x="193.04" y="88.9" size="1.778" layer="96" display="off"/>
+<attribute name="MANF2" x="193.04" y="88.9" size="1.778" layer="96" display="off"/>
+<attribute name="MANF2#" x="193.04" y="88.9" size="1.778" layer="96" display="off"/>
 </instance>
 </instances>
