File: nephelometer/circuitry/band-motor-teensy.brd (EAGLE design)
At the start: 73 x 55 mm, 37 parts, among them IC1 7805TV, J1 PJ-102A, J2 MotA, J3 AUDIO-JACK2PTH, J4 RJ11-6PTH, J5 MotA, J6 AUDIO-JACK2PTH, T1 2N2222, T2 2N2222

Commit message: Revised detector board circuit, picked filter values, finalized parts
Parts:
- R11, R6: value 150R -> 330R
