File: nephelometer/circuitry/band-dsp-teensy.sch (EAGLE design)
At the start: 42 parts, among them IC1 LM4041CILP, IC2 AD822N, IC3 MCP6S21, J1 RJ11-6PTH, Q1 IRLB8721, T1 2N2222, T2 2N2222

Commit message: Separate 3V3 supply for analog circuits. Guard ring for TIA
Parts:
- added C10: 1µF, adafruit:C-US025-030X050
- added IC4: LP2950ACZ-3.3, v-reg:LP2950ACZ-3.3
- C3: device adafruit:C-US050-024X044 -> adafruit:C-US025-025X050
- C8: device adafruit:C-US025-030X050 -> adafruit:CPOL-USE2.5-5; DIGIKEY# 445-8348-ND -> 478-8042-1-ND; MANF TDK Corporation -> AVX Corporation; MANF# FK16X7R1C106K -> TAP106K016SRW
Connections:
- new net N$2: BRD1.3.3V, R14.1
- net +3V3: now also C8.+, IC4.OUT; no longer BRD1.3.3V, C8.1, R14.1
- net +5V: now also C10.1, IC4.IN
- net GND: now also C10.2, C8.-, IC4.GND; no longer C8.2
Other:
- note added: "Separate 3.3V for analog"
- moved on the sheet: AGND
