File: nephelometer/circuitry/band-dsp-feather.sch (EAGLE design)
At the start: 44 parts, among them IC1 LM4041CILP, IC2 AD822N, IC3 MCP6S21, IC4 LP2950ACZ-3.3, J1 RJ11-6PTH, Q1 IRLB8721, T1 2N2222, T2 2N2222

Commit message: Feather-based board with external ADC
Parts:
- removed 1V65, BPF, TIA: TPTP10R, testpad:TPTP10R
- removed AGND: (no value), adafruit:PINHD-1X1
- removed BRD1: TEENSY_3.1-3.2_DIL+4, Teensy_3_and_LC_Series_Boards_v1.4:TEENSY_3.1-3.2_DIL+4
- removed EMIT: TPPAD1-13, testpad:TPPAD1-13
- removed LED2: LED3MM_WP937EGW, ingolia:LED3MM_WP937EGW
- removed U$5: LED3MM_H101C, ingolia:LED3MM_H101C
- added C11, C14: 1.2nF, adafruit:C-US025-025X050
- added C12: 100nF, adafruit:C-US025-025X050
- added C13: 1uF, adafruit:C-US025-025X050
- added D3, D4, D5, D6: (no value), diode:ZENER-DIODEF126-10
- added LD1: (no value), led:DUOLED-RG-C
- added R15, R16: 1k5, adafruit:R-US_0207/9
- added R17, R19, R21, R23: 1K0, adafruit:R-US_0207/9
- added R18, R20, R22, R24: 33K, adafruit:R-US_0207/9
- added R25: 470R, adafruit:R-US_0207/9
- added R6: 3K3, adafruit:R-US_0207/9
- added T3, T4, T5, T6: 2N2222, adafruit:2N2222
- added U$7: FEATHER_M0, ingolia:FEATHER_M0
- added U$8: MAX144, ingolia:MAX144
- D2: value 1N5817-T -> (none); device diode:1N5817-T -> diode:ZENER-DIODEF126-10; DIGIKEY# 1N5817FSCT-ND -> (none); MANF Fairchild Semiconductor -> (none); MANF# 1N5817 -> (none)
- Q1: device ingolia:IRLB8721HORIZONTAL -> transistor-small-signal:BS170
- R11, R9: value 4K7 -> 10K
- R12: value 330R -> 470R
- R13: DIGIKEY# CF14JT330RCT-ND -> 6.65KXBK-ND; MANF Stackpole Electronics Inc. -> Yageo; MANF# CF14JT330R -> MFR-25FBF52-6K65
- R14: value 330R -> 470R; device adafruit:R-US_0207/9 -> adafruit:R-US_0207/5V
Connections:
- net N$1 renamed FB
- removed net LEDCTRL: R11.2, T2.B
- removed net N$12: LED2.GK, R12.2
- removed net V+: BRD1.VUSB, D2.A
- new net BPF: C6.2, IC2B.OUT, IC3.IN+, R10.2
- new net CS_ADC: U$7.6, U$8.SHDN
- new net LED_CTRL: R15.2, R16.1, U$7.A3/17
- new net MISO: U$7.MISO/22, U$8.DOUT
- new net MOT1_CTRL: T3.E, U$7.A4/18
- new net MOT2_CTRL: T4.E, U$7.A5/19
- new net MOT3: D6.C, J1.6, R21.2
- new net MOT3_CTRL: T5.E, U$7.10
- new net MOT4: D5.C, J1.1, R23.2
- new net MOT4_CTRL: T6.E, U$7.11
- new net N$1: R19.1, T4.C
- new net N$13: R11.1, R6.1, T1.B
- new net N$15: C11.2, R11.2, R15.1
- new net N$16: R16.2, T2.B
- new net N$19: R17.1, T3.C
- new net N$20: R18.2, T3.B
- new net N$21: R24.2, T6.B
- new net N$23: C14.1, R13.1, U$8.CH0, U$8.CH1
- new net TIA: C2.2, IC2A.OUT, R4.2, R8.2
- new net VDD: R18.1, R20.1, R22.1, R24.1, U$7.3V3
- new net VEXT: D1.A, D2.C, J1.5, R12.2
- net +3V3: now also C12.2, C13.2, U$8.REF, U$8.VDD; no longer BRD1.AREF
- net +5V: now also R14.1, R25.2, U$7.VBUS; no longer BRD1.VIN, D2.C, U$5.A
- net 1V65: no longer 1V65.TP, BRD1.A11
- net CS_PGA: now also U$7.5; no longer BRD1.15/A1/T
- net GND: now also C11.1, C12.1, C13.1, C14.2, D2.A, D3.A, D4.A, D5.A, D6.A, LD1.C, U$6.K, U$7.GND, U$8.GND; no longer AGND.1, BRD1.AGND, BRD1.GND, R12.1, R13.1
- net MOSI: now also U$7.MOSI/23; no longer BRD1.11/MOSI
- net MOT1: now also D3.C, R17.2; no longer BRD1.16/A2/T
- net MOT2: now also D4.C, R19.2; no longer BRD1.17/A3/T
- net N$10: now also R23.1, T6.C; no longer D1.A, J1.5, LED2.GA
- net N$11: now also T2.C
- net N$14: now also R6.2; no longer T1.B
- net N$2: now also R20.2, T4.B; no longer BRD1.3.3V, R14.1
- net N$22: now also LD1.AR, R12.1; no longer C2.2, IC2A.OUT, R4.2, R8.2, TIA.TP
- net N$4: now also R13.2; no longer BRD1.A10
- net N$5: now also R21.1, T5.C; no longer BRD1.2, EMIT.TP, R11.1, U$6.K
- net N$6: now also R22.2, T5.B; no longer BPF.TP, C6.2, IC2B.OUT, IC3.IN+, R10.2
- net N$7: now also LD1.AG, R25.1; no longer R13.2, U$5.K
- net N$8: no longer T2.C
- net SCK: now also U$7.SCK/24, U$8.SCLK; no longer BRD1.13/SCK/LED
Other:
- note added: "SPI Analog-to-Digital"
- moved on the sheet: C1, C10, C3, C5, C7, C8, C9, D1, IC1, IC2P, IC3, IC4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
