File: nephelometer/circuitry/band-motor-feather.brd (EAGLE design)
At the start: 95 x 55 mm, 74 parts, among them IC1 7805TV, IC2 L293D, J1 PJ-102A, J10 MotA, J2 MotA, J3 AUDIO-JACK2PTH, J4 RJ11-6PTH, J5 MotA, J6 AUDIO-JACK2PTH, J7 MotA, J8 MotA, J9 MotA, T1 2N2222, T2 2N2222, T3 2N2222, T4 2N2222, T5 2N2222, T6 2N2222

Commit message: Finalized Feather nephelometer with separate ADC and 4 robust motor controls
Parts:
- removed J7, J8: MotA, ingolia:1X02_3.5MM_MOT
- removed R24: 10K, adafruit:0207/10
- added J109, J110: MotA, ingolia:1X02_3.5MM_MOT
- added R124: 10K, adafruit:0207/10
- C105: value (none) -> 1µF
- C106: value (none) -> 100nF
- R105, R106, R107, R108: value 10K -> 4K7
- renumbered C1 to C101, C2 to C102, C3 to C103, C4 to C104, C5 to C105, C6 to C106, D1 to D110, D10 to D101, D2 to D104, D3 to D103, D4 to D109, D5 to D108, D6 to D107, D7 to D106, D8 to D105, D9 to D102, IC1 to IC101, IC2 to IC102, J1 to J108, J10 to J104, J2 to J107, J3 to J102, J4 to J103, J5 to J106, J6 to J101, J9 to J105, LED1 to LED105, LED2 to LED104, LED3 to LED103, LED4 to LED102, LED5 to LED101, MCU1 to IC103, Q1 to Q104, Q2 to Q103, Q3 to Q102, Q4 to Q101, R1 to R121, R10 to R116, R11 to R117, R12 to R106, R13 to R112, R14 to R113, R15 to R114, R16 to R105, R17 to R109, R18 to R110, R19 to R111, R2 to R118, R20 to R122, R21 to R123, R22 to R126, R23 to R125, R25 to R102, R26 to R101, R3 to R119, R4 to R108, R5 to R120, R6 to R104, R7 to R103, R8 to R107, R9 to R115, T1 to T104, T2 to T103, T3 to T102, T4 to T101, T5 to T105, T6 to T106
Connections:
- net +5V: now also R124.2; no longer R24.2
- net EN: now also R124.1; no longer R24.1
- net N$15: now also J109.1A; no longer J7.1A
- net N$16: now also J109.2K; no longer J7.2K
- net N$18: now also J110.2K; no longer J8.2K
- net N$19: now also J110.1A; no longer J8.1A
Routing:
- net N$11: track 27.9 -> 18.5 mm
- net N$19: track 15.7 -> 24.3 mm
- net N$15: track 11.2 -> 16.2 mm
- net EN: track 39.7 -> 44.2 mm
- net +5V: track 193.2 -> 195.7 mm
- net N$16: track 14.3 -> 16.4 mm
- net N$18: track 14.6 -> 13.5 mm
Other:
- board text added: "band-motor-feather ingolia@ berkeley.edu 17-06-06"
- board text removed: "band-motor-teensy ingolia@berkeley.edu 16-11-30"

Commit message: Minor updates after test assembly
Other:
- board text added: "band-motor-feather ingolia@ berkeley.edu 17-06-22"
- board text removed: "band-motor-feather ingolia@ berkeley.edu 17-06-06"
Changed lines of the file:
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@@
 ingolia@
       berkeley.edu
-17-06-06</text>
+17-06-22</text>
 </plain>
 <attributes>
@@
 </element>
 <element name="D109" library="diode" package="F126Z10" value="" x="87" y="7" smashed="yes">
-<attribute name="DIGIKEY#" value="SA12CALFCT-ND" x="87" y="7" size="1.778" layer="27" display="off"/>
+<attribute name="DIGIKEY#" value="SA12ALFCT-ND" x="87" y="7" size="1.778" layer="27" display="off"/>
 <attribute name="MANF" value="Littelfuse Inc." x="87" y="7" size="1.778" layer="27" display="off"/>
-<attribute name="MANF#" value="SA12CA" x="87" y="7" size="1.778" layer="27" display="off"/>
+<attribute name="MANF#" value="SA12A" x="87" y="7" size="1.778" layer="27" display="off"/>
 <attribute name="NAME" x="82.722" y="8.325" size="1.27" layer="25" ratio="10" rot="R90"/>
 <attribute name="VALUE" x="83.825" y="3.952" size="1.27" layer="27" ratio="10"/>
@@
 <attribute name="MANF" value="Stackpole Electronics Inc" x="40" y="18.5" size="1.778" layer="27" rot="R90" display="off"/>
 <attribute name="MANF#" value="CF14JT10K0" x="40" y="18.5" size="1.778" layer="27" rot="R90" display="off"/>
-<attribute name="NAME" x="24.476" y="15.452" size="1.27" layer="25" ratio="10" rot="R90"/>
+<attribute name="NAME" x="29.976" y="14.452" size="1.27" layer="25" ratio="10" rot="R90"/>
 <attribute name="VALUE" x="28.135" y="16.2394" size="1.27" layer="27" ratio="10" rot="R90"/>
 </element>
@@
 <attribute name="MANF" value="Stackpole Electronics Inc" x="28" y="17" size="1.778" layer="27" rot="R270" display="off"/>
 <attribute name="MANF#" value="CF14JT330R" x="28" y="17" size="1.778" layer="27" rot="R270" display="off"/>
-<attribute name="NAME" x="29.024" y="18.048" size="1.27" layer="25" ratio="10" rot="R270"/>
+<attribute name="NAME" x="23.524" y="11.048" size="1.27" layer="25" ratio="10" rot="R270"/>
 <attribute name="VALUE" x="23.365" y="19.2606" size="1.27" layer="27" ratio="10" rot="R270"/>
 </element>
